File: STM32_2CH_Dimmer.sch (KiCad schematic (older format))
At the start: 33 parts, among them J1 Power, J2 Encoder1, J3 Encoder2, J4 LED1, J5 LED2, Q1 IRF3708, Q2 IRF3708, SW1 Config, U1 173950378, U2 DS18B20, U3 STM32F103Generic, U4 AT24CS32, U5 CC1101

Commit message: update
Parts:
- C7: footprint Capacitor_SMD:C_0603_1608Metric_Pad1.05x0.95mm_HandSolder -> Capacitor_SMD:C_0805_2012Metric_Pad1.15x1.40mm_HandSolder
- Q1, Q2: footprint TO_SOT_Packages_THT:TO-220_Vertical -> Package_TO_SOT_THT:TO-220-3_Vertical
Changed lines of the file:
@@
 F 0 "C7" H 8210 1620 50  0000 L CNN
 F 1 "100n" H 8210 1470 50  0000 L CNN
-F 2 "Capacitor_SMD:C_0603_1608Metric_Pad1.05x0.95mm_HandSolder" H 8200 1550 50  0001 C CNN
+F 2 "Capacitor_SMD:C_0805_2012Metric_Pad1.15x1.40mm_HandSolder" H 8200 1550 50  0001 C CNN
 F 3 "" H 8200 1550 50  0001 C CNN
 	1    8200 1550
@@
 F 0 "Q1" H 9850 3700 50  0000 L CNN
 F 1 "IRF3708" H 9850 3800 50  0000 L CNN
-F 2 "TO_SOT_Packages_THT:TO-220_Vertical" H 9900 3725 50  0001 L CIN
+F 2 "Package_TO_SOT_THT:TO-220-3_Vertical" H 9900 3725 50  0001 L CIN
 F 3 "" H 9650 3800 50  0001 L CNN
 	1    9650 3800
@@
 F 0 "Q2" H 9850 5000 50  0000 L CNN
 F 1 "IRF3708" H 9850 5100 50  0000 L CNN
-F 2 "TO_SOT_Packages_THT:TO-220_Vertical" H 9900 5025 50  0001 L CIN
+F 2 "Package_TO_SOT_THT:TO-220-3_Vertical" H 9900 5025 50  0001 L CIN
 F 3 "" H 9650 5100 50  0001 L CNN
 	1    9650 5100

Commit message: V1.1
Parts:
- added C1: 10µ, Capacitor_SMD:C_1210_3225Metric_Pad1.42x2.65mm_HandSolder, symbol STM32_2CH_Dimmer-rescue:C_Small-STM32Dimmer-rescue
- C2: renamed from C5; value 10µ -> 22µ
- C8: renamed from C6; footprint Capacitor_SMD:C_0603_1608Metric_Pad1.05x0.95mm_HandSolder -> Capacitor_SMD:C_0805_2012Metric_Pad1.15x1.40mm_HandSolder
- U1: value 173950378 -> LC78
- renumbered C7 to C3, C1 to C4, C3 to C5, C2 to C6, C4 to C7, J4 to J2, J2 to J3, J3 to J4, R5 to R1, R9 to R10, R6 to R2, R7 to R3, R1 to R4, R2 to R5, R8 to R6, R10 to R7, R3 to R8, R4 to R9, U3 to U2, U5 to U3, U2 to U5
Connections:
- wire segments 149 -> 152
Other:
- moved on the sheet: C2, C3, U1, U3

Commit message: V1.2
Parts:
- U1: value LC78 -> LC78_03-05
Other:
- note added: "CC BY-NC-SA 4.0"
- note added: "use SS15/SS16 Schottky @ 24V"
Changed lines of the file:
@@
 Title "HM_STM32_2CH_Dimmer"
 Date ""
-Rev "V1.1"
+Rev "V1.2"
 Comp ""
 Comment1 ""
@@
 P 1950 1100
 F 0 "U1" H 1950 1375 50  0000 C CNN
-F 1 "LC78" H 1950 1284 50  0000 C CNN
+F 1 "LC78_03-05" H 1950 1284 50  0000 C CNN
 F 2 "Homebrew:WE_FDSM_173950378" H 1950 1100 50  0001 C CNN
-F 3 "" H 1950 1100 50  0001 C CNN
+F 3 "https://www.reichelt.de/dc-dc-wandler-1-65-w-3-3-v-500-ma-to-220-lc78-03-0-5-p242822.html" H 1950 1100 50  0001 C CNN
 	1    1950 1100
 	1    0    0    -1
@@
 Wire Wire Line
 	1450 1700 1450 1550
+Text Notes 7975 6925 0    157  ~ 31
+CC BY-NC-SA 4.0
+Text Notes 8200 4450 0    50   ~ 0
+use SS15/SS16 Schottky @ 24V
 $EndSCHEMATC

Commit message: V1.2
Parts:
- U1: footprint Homebrew:WE_FDSM_173950378 -> Homebrew:LC78_03-05
Changed lines of the file:
@@
 F 1 "SS14" H 9550 3350 50  0000 C CNN
 F 2 "Diodes_SMD:D_SMA" H 9550 3450 50  0001 C CNN
-F 3 "https://de.aliexpress.com/item/100PCS-SMA-Rectifier-diode-1N5819-SS14-1N5822-SS34-SR160-SS16-1N5817-SS12-SR1100-SS110-SR360-SS36/32849859393.html?spm=a2g0x.search0104.3.1.51e17831k6mqUy&ws_ab_test=searchweb0_0,searchweb201602_1_10320_10152_10321_10151_10065_10344_10068_10342_10547_10343_10322_10340_10548_10341_10696_10084_10083_10618_10304_10307_10820_10821_5011711_5723611_10302_5011811_10843_10059_100031_10319_10103_10624_10623_10622_10621_10620,searchweb201603_55,ppcSwitch_5&algo_expid=9582c958-26fb-4969-b9f2-a0d34c9e4af6-0&algo_pvid=9582c958-26fb-4969-b9f2-a0d34c9e4af6&transAbTest=ae803_1&priceBeautifyAB=0" H 9550 3450 50  0001 C CNN
+F 3 "https://de.aliexpress.com/item/100PCS-SMA-Rectifier-diode-1N5819-SS14-1N5822-SS34-SR160-SS16-1N5817-SS12-SR1100-SS110-SR360-SS36/32849859393.html" H 9550 3450 50  0001 C CNN
 	1    9550 3450
 	-1   0    0    1
@@
 F 1 "SS14" H 9550 4650 50  0000 C CNN
 F 2 "Diodes_SMD:D_SMA" H 9550 4750 50  0001 C CNN
-F 3 "https://de.aliexpress.com/item/100PCS-SMA-Rectifier-diode-1N5819-SS14-1N5822-SS34-SR160-SS16-1N5817-SS12-SR1100-SS110-SR360-SS36/32849859393.html?spm=a2g0x.search0104.3.1.51e17831k6mqUy&ws_ab_test=searchweb0_0,searchweb201602_1_10320_10152_10321_10151_10065_10344_10068_10342_10547_10343_10322_10340_10548_10341_10696_10084_10083_10618_10304_10307_10820_10821_5011711_5723611_10302_5011811_10843_10059_100031_10319_10103_10624_10623_10622_10621_10620,searchweb201603_55,ppcSwitch_5&algo_expid=9582c958-26fb-4969-b9f2-a0d34c9e4af6-0&algo_pvid=9582c958-26fb-4969-b9f2-a0d34c9e4af6&transAbTest=ae803_1&priceBeautifyAB=0" H 9550 4750 50  0001 C CNN
+F 3 "https://de.aliexpress.com/item/100PCS-SMA-Rectifier-diode-1N5819-SS14-1N5822-SS34-SR160-SS16-1N5817-SS12-SR1100-SS110-SR360-SS36/32849859393.html" H 9550 4750 50  0001 C CNN
 	1    9550 4750
 	-1   0    0    1
@@
 F 0 "U1" H 1950 1375 50  0000 C CNN
 F 1 "LC78_03-05" H 1950 1284 50  0000 C CNN
-F 2 "Homebrew:WE_FDSM_173950378" H 1950 1100 50  0001 C CNN
+F 2 "Homebrew:LC78_03-05" H 1950 1100 50  0001 C CNN
 F 3 "https://www.reichelt.de/dc-dc-wandler-1-65-w-3-3-v-500-ma-to-220-lc78-03-0-5-p242822.html" H 1950 1100 50  0001 C CNN
 	1    1950 1100
